Commit message: refactor: move JinBot workflow to IsaacLab

File: robot/robot.urdf (robot description, URDF)
Before this commit: robot robot, 15 links, 14 joints
Links:
- removed link closing_leg2_ball_1
- removed link closing_leg2_ball_2
- removed link closing_leg3_ball_1
- removed link closing_leg3_ball_2
- removed link leg1_ball_y_link
- removed link leg1_ball_z_link
- removed link leg1_lower
- removed link leg1_upper
- removed link leg2_lower
- removed link leg2_upper
- removed link leg3_lower
- removed link leg3_upper
- removed link platform
- removed link tracking
- added link l_ankle_pitch_link, mass 0.20135; collision mesh filename=assets/part_1__4.stl; visual mesh filename=assets/part_1__4.stl
- added link l_hip_pitch_link, mass 1.70514; collision mesh filename=assets/dm_j8006_2ec_v1_1__2.stl; collision mesh filename=assets/dm_j8006_2ec_v1_1__3.stl
- added link l_hip_roll_link, mass 0.127662; collision mesh filename=assets/part_1__2.stl; visual mesh filename=assets/part_1__2.stl
- added link l_hip_yaw_link, mass 0.784517; collision mesh filename=assets/dm_j8006_2ec_v1_1.stl; collision mesh filename=assets/part_1.stl
- added link l_knee_pitch_link, mass 0.6749; collision mesh filename=assets/dm_j6006_2ec.stl; collision mesh filename=assets/part_2__3.stl
- added link r_ankle_pitch_link, mass 0.20135; collision mesh filename=assets/part_1__4.stl; visual mesh filename=assets/part_1__4.stl
- added link r_hip_pitch_link, mass 1.70514; collision mesh filename=assets/dm_j8006_2ec_v1_1__2.stl; collision mesh filename=assets/dm_j8006_2ec_v1_1__3.stl
- added link r_hip_roll_link, mass 0.127662; collision mesh filename=assets/part_1__2.stl; visual mesh filename=assets/part_1__2.stl
- added link r_hip_yaw_link, mass 0.784517; collision mesh filename=assets/dm_j8006_2ec_v1_1.stl; collision mesh filename=assets/part_1.stl
- added link r_knee_pitch_link, mass 0.6749; collision mesh filename=assets/dm_j6006_2ec.stl; collision mesh filename=assets/part_2__3.stl
- link base_link: mass 0.701657 -> 1.47836; geometry collision mesh filename=assets/dm_j8006_2ec_v1_1.stl; collision mesh filename=assets/dm_j8006_2ec_v1_1.stl
Joints:
- removed joint closing_leg2_ball_1_frame
- removed joint closing_leg2_ball_2_frame
- removed joint closing_leg3_ball_1_frame
- removed joint closing_leg3_ball_2_frame
- removed joint leg1_1
- removed joint leg1_2
- removed joint leg1_ball_x
- removed joint leg1_ball_y
- removed joint leg1_ball_z
- removed joint leg2_1
- removed joint leg2_2
- removed joint leg3_1
- removed joint leg3_2
- removed joint tracking_frame
- added joint l_ankle_pitch: type revolute, parent l_knee_pitch_link, child l_ankle_pitch_link, origin xyz=6.85453e-05 0.160119 0.0195 rpy=0 -0 -0, axis 0 0 1, limit lower=-0.523599 upper=0.523599 effort=10 velocity=10
- added joint l_hip_pitch: type revolute, parent l_hip_roll_link, child l_hip_pitch_link, origin xyz=0.082 5.91774e-05 0.00460127 rpy=3.14159 -1.5708 0, axis 0 0 1, limit lower=-0.523599 upper=0.872665 effort=10 velocity=10
- added joint l_hip_roll: type revolute, parent l_hip_yaw_link, child l_hip_roll_link, origin xyz=0.0195 -0.000905374 -0.071579 rpy=1.5708 -0 1.5708, axis 0 0 1, limit lower=-0.349066 upper=0.349066 effort=10 velocity=10
- added joint l_hip_yaw: type revolute, parent base_link, child l_hip_yaw_link, origin xyz=0.000993584 0.0599212 -0.0215 rpy=0 0 0, axis 0 0 1, limit lower=-0.523599 upper=0.523599 effort=10 velocity=10
- added joint l_knee_pitch: type revolute, parent l_hip_pitch_link, child l_knee_pitch_link, origin xyz=-0 0.12 -0 rpy=-0 0 0, axis 0 0 1, limit lower=-1.74533 upper=0 effort=10 velocity=10
- added joint r_ankle_pitch: type revolute, parent r_knee_pitch_link, child r_ankle_pitch_link, origin xyz=6.85453e-05 -0.160119 0.0195 rpy=0 0 0, axis 0 0 1, limit lower=-0.523599 upper=0.523599 effort=10 velocity=10
- added joint r_hip_pitch: type revolute, parent r_hip_roll_link, child r_hip_pitch_link, origin xyz=-0.082 -5.91774e-05 0.00460127 rpy=-0 -1.5708 0, axis 0 0 1, limit lower=-0.872665 upper=0.523599 effort=10 velocity=10
- added joint r_hip_roll: type revolute, parent r_hip_yaw_link, child r_hip_roll_link, origin xyz=0.0195 0 -0.0715 rpy=1.5708 0 1.5708, axis 0 0 1, limit lower=-0.349066 upper=0.349066 effort=10 velocity=10
- added joint r_hip_yaw: type revolute, parent base_link, child r_hip_yaw_link, origin xyz=0.000993584 -0.0600788 -0.0215 rpy=0 0 0, axis 0 0 1, limit lower=-0.523599 upper=0.523599 effort=10 velocity=10
- added joint r_knee_pitch: type revolute, parent r_hip_pitch_link, child r_knee_pitch_link, origin xyz=-0 -0.12 0 rpy=0 -0 0, axis 0 0 1, limit lower=0 upper=1.74533 effort=10 velocity=10
